File: multicartridge-smd/p2000t-multicartridge-smd/p2000t-multicartridge-smd.kicad_pcb (KiCad board)
At the start: 2 copper layers, 80 x 100 mm, 25 parts, among them J1 P2000T_cartridge_edge, SW1 Soft Reset, SW2 SW_DIP_x05, U1 SST39SF040, U2 74HC123, U3 74HC00

Commit message: Completing PCB
Parts:
- added G2: LOGO, libs:qrcode, B.Cu at (105.9, 110.1)
- TP4: value PB_~NMI~ -> PB_~{NMI}
- moved JP1 27.2 mm to (99.5, 89.8), turned to 180 degrees
- moved R3 16.4 mm to (96.6, 80.6), turned to -90 degrees
- moved R2 10.8 mm to (82.7, 67.4), turned to -90 degrees
- moved C3 8.14 mm to (90.3, 66.4), turned to 0 degrees
- moved C5 5.46 mm to (75.1, 66.9)
- moved C4 4.49 mm to (96.6, 76.8)
- moved U3 4.06 mm to (75.1, 74.3)
- moved U2 3.93 mm to (90.3, 74.2)
- moved C1 3.41 mm to (82.7, 72.0)
- renumbered G*** to G1
Routing:
- net GND: track 0.00 -> 252.9 mm, vias 0 -> 2
- net +5V: track 0.00 -> 229.3 mm, vias 0 -> 3
- net A12C: track 0.00 -> 150.3 mm
- net ~{CARSEL1}: track 0.00 -> 141.8 mm, vias 0 -> 2
- net ~{CARSEL2}: track 0.00 -> 93.3 mm, vias 0 -> 1
- net ~{NMI}: track 0.00 -> 91.7 mm, vias 0 -> 1
- net Net-(R1-Pad2): track 0.00 -> 81.8 mm, vias 0 -> 1
- net A14: track 0.00 -> 70.4 mm
- net D3: track 0.00 -> 60.3 mm, vias 0 -> 1
- net A8: track 0.00 -> 59.8 mm
- net A11: track 0.00 -> 59.7 mm, vias 0 -> 3
- net D5: track 0.00 -> 59.0 mm
- net A6: track 0.00 -> 55.4 mm, vias 0 -> 2
- net A7: track 0.00 -> 53.3 mm, vias 0 -> 1
- net D0: track 0.00 -> 53.1 mm, vias 0 -> 2
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Other:
- board size 80 x 100 mm -> 80 x 100.3 mm
