File: multicartridge-smd/p2000t-multicartridge-smd/p2000t-multicartridge-smd.kicad_sch (KiCad schematic)
At the start: 24 parts, among them J1 P2000T_cartridge_edge, SW1 Soft Reset, SW2 SW_DIP_x05, U1 SST39SF040, U2 74HC123, U3 74HC00

Commit message: Completing PCB
Parts:
- TP4: value PB_~NMI~ -> PB_~{NMI}
- U2: JLCPCB (none) -> C5597
- U3: JLCPCB (none) -> C5586
Other:
- title: P2000T Multirom Cartridge -> P2000T Multirom Cartridge (SMD)
Changed lines of the file:
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@@
   (paper "A4")
   (title_block
-    (title "P2000T Multirom Cartridge")
-    (date "2021-08-14")
+    (title "P2000T Multirom Cartridge (SMD)")
+    (date "2023-09-15")
     (rev "1")
   )
@@
       (effects (font (size 1.27 1.27)) hide)
     )
+    (property "JLCPCB" "C5586" (id 4) (at 129.54 39.37 0)
+      (effects (font (size 1.27 1.27)) hide)
+    )
     (pin "1")
     (pin "2")
@@
       (effects (font (size 1.27 1.27)) hide)
     )
+    (property "JLCPCB" "C5586" (id 4) (at 109.22 54.61 0)
+      (effects (font (size 1.27 1.27)) hide)
+    )
     (pin "1")
     (pin "2")
@@
       (effects (font (size 1.27 1.27)) hide)
     )
+    (property "JLCPCB" "C5586" (id 4) (at 109.22 68.58 0)
+      (effects (font (size 1.27 1.27)) hide)
+    )
     (pin "1")
     (pin "2")
@@
       (effects (font (size 1.27 1.27)) hide)
     )
+    (property "JLCPCB" "C5586" (id 4) (at 109.22 39.37 0)
+      (effects (font (size 1.27 1.27)) hide)
+    )
     (pin "1")
     (pin "2")
@@
       (effects (font (size 1.27 1.27)) hide)
     )
+    (property "JLCPCB" "C5586" (id 4) (at 118.11 86.36 0)
+      (effects (font (size 1.27 1.27)) hide)
+    )
     (pin "1")
     (pin "2")
@@
     )
     (property "Datasheet" "https://assets.nexperia.com/documents/data-sheet/74HC_HCT123.pdf" (id 3) (at 72.39 144.78 0)
+      (effects (font (size 1.27 1.27)) hide)
+    )
+    (property "JLCPCB" "C5597" (id 4) (at 72.39 144.78 0)
       (effects (font (size 1.27 1.27)) hide)
     )
@@
       (effects (font (size 1.27 1.27)) hide)
     )
+    (property "JLCPCB" "C5597" (id 4) (at 72.39 172.72 0)
+      (effects (font (size 1.27 1.27)) hide)
+    )
     (pin "1")
     (pin "13")
@@
       (effects (font (size 1.27 1.27)) hide)
     )
+    (property "JLCPCB" "C5597" (id 4) (at 118.11 144.78 0)
+      (effects (font (size 1.27 1.27)) hide)
+    )
     (pin "1")
     (pin "13")
@@
       (effects (font (size 1.27 1.27)) (justify left))
     )
-    (property "Value" "PB_~NMI~" (id 1) (at 243.9162 144.5514 0)
+    (property "Value" "PB_~{NMI}" (id 1) (at 243.9162 144.5514 0)
       (effects (font (size 1.27 1.27)) (justify left))
     )
@@
     )
     (path "/00000000-0000-0000-0000-00006132c376"
-      (reference "TP4") (unit 1) (value "PB_~NMI~") (footprint "TestPoint:TestPoint_THTPad_D1.5mm_Drill0.7mm")
+      (reference "TP4") (unit 1) (value "PB_~{NMI}") (footprint "TestPoint:TestPoint_THTPad_D1.5mm_Drill0.7mm")
     )
     (path "/00000000-0000-0000-0000-000060ffad49"

Commit message: Updating schematic
Parts:
- C1: LCSC (none) -> C16133
- C2, C3, C5: LCSC (none) -> C49678
- C4: LCSC (none) -> C28323
- R1, R3, R4, R5, R6, R7, R8: LCSC (none) -> C17414
- R2: LCSC (none) -> C17713
- U2: LCSC (none) -> C5597
- U3: LCSC (none) -> C5586
Changed lines of the file:
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@@
+      (effects (font (size 1.27 1.27)) hide)
+    )
+    (property "LCSC" "C49678" (id 5) (at 57.15 29.21 0)
       (effects (font (size 1.27 1.27)) hide)
     )
@@
       (effects (font (size 1.27 1.27)) hide)
     )
+    (property "LCSC" "C5586" (id 5) (at 129.54 39.37 0)
+      (effects (font (size 1.27 1.27)) hide)
+    )
     (pin "1")
     (pin "2")
@@
       (effects (font (size 1.27 1.27)) hide)
     )
+    (property "LCSC" "C5586" (id 5) (at 109.22 54.61 0)
+      (effects (font (size 1.27 1.27)) hide)
+    )
     (pin "1")
     (pin "2")
@@
       (effects (font (size 1.27 1.27)) hide)
     )
+    (property "LCSC" "C5586" (id 5) (at 109.22 68.58 0)
+      (effects (font (size 1.27 1.27)) hide)
+    )
     (pin "1")
     (pin "2")
@@
       (effects (font (size 1.27 1.27)) hide)
     )
+    (property "LCSC" "C5586" (id 5) (at 109.22 39.37 0)
+      (effects (font (size 1.27 1.27)) hide)
+    )
     (pin "1")
     (pin "2")
@@
       (effects (font (size 1.27 1.27)) hide)
     )
+    (property "LCSC" "C5586" (id 5) (at 118.11 86.36 0)
+      (effects (font (size 1.27 1.27)) hide)
+    )
     (pin "1")
     (pin "2")
@@
       (effects (font (size 1.27 1.27)) hide)
     )
+    (property "LCSC" "C49678" (id 5) (at 118.11 100.33 0)
+      (effects (font (size 1.27 1.27)) hide)
+    )
     (pin "1")
     (pin "2")
@@
     )
     (property "JLCPCB" "C5597" (id 4) (at 72.39 144.78 0)
+      (effects (font (size 1.27 1.27)) hide)
+    )
+    (property "LCSC" "C5597" (id 5) (at 72.39 144.78 0)
       (effects (font (size 1.27 1.27)) hide)
     )
@@
       (effects (font (size 1.27 1.27)) hide)
     )
+    (property "LCSC" "C5597" (id 5) (at 72.39 172.72 0)
+      (effects (font (size 1.27 1.27)) hide)
+    )
     (pin "1")
     (pin "13")
@@
       (effects (font (size 1.27 1.27)) hide)
     )
+    (property "LCSC" "C49678" (id 5) (at 72.39 186.69 0)
+      (effects (font (size 1.27 1.27)) hide)
+    )
     (pin "1")
     (pin "2")
@@
     )
     (property "JLCPCB" "C5597" (id 4) (at 118.11 144.78 0)
+      (effects (font (size 1.27 1.27)) hide)
+    )
+    (property "LCSC" "C5597" (id 5) (at 118.11 144.78 0)
       (effects (font (size 1.27 1.27)) hide)
     )
@@
       (effects (font (size 1.27 1.27)) hide)
     )
+    (property "LCSC" "C17414" (id 5) (at 40.64 138.43 0)
+      (effects (font (size 1.27 1.27)) hide)
+    )
     (pin "1")
     (pin "2")
@@
       (effects (font (size 1.27 1.27)) hide)
     )
+    (property "LCSC" "C17713" (id 5) (at 58.42 129.54 0)
+      (effects (font (size 1.27 1.27)) hide)
+    )
     (pin "1")
     (pin "2")
@@
     )
     (property "JLCPCB" "C16133" (id 4) (at 49.53 140.97 0)
+      (effects (font (size 1.27 1.27)) hide)
+    )
+    (property "LCSC" "C16133" (id 5) (at 49.53 140.97 0)
       (effects (font (size 1.27 1.27)) hide)
     )
@@
       (effects (font (size 1.27 1.27)) hide)
     )
+    (property "LCSC" "C17414" (id 5) (at 91.44 134.62 0)
+      (effects (font (size 1.27 1.27)) hide)
+    )
     (pin "1")
     (pin "2")
@@
       (effects (font (size 1.27 1.27)) hide)
     )
+    (property "LCSC" "C28323" (id 5) (at 97.79 140.97 0)
+      (effects (font (size 1.27 1.27)) hide)
+    )
     (pin "1")
     (pin "2")
@@
     )
     (property "JLCPCB" "C17414" (id 4) (at 250.19 52.07 0)
+      (effects (font (size 1.27 1.27)) hide)
+    )
+    (property "LCSC" "C17414" (id 5) (at 250.19 52.07 0)
       (effects (font (size 1.27 1.27)) hide)
     )
@@
       (effects (font (size 1.27 1.27)) hide)
     )
+    (property "LCSC" "C17414" (id 5) (at 255.27 38.735 0)
+      (effects (font (size 1.27 1.27)) hide)
+    )
     (pin "1")
     (pin "2")
@@
       (effects (font (size 1.27 1.27)) hide)
     )
+    (property "LCSC" "C17414" (id 5) (at 260.35 52.07 0)
+      (effects (font (size 1.27 1.27)) hide)
+    )
     (pin "1")
     (pin "2")
@@
       (effects (font (size 1.27 1.27)) hide)
     )
+    (property "LCSC" "C17414" (id 5) (at 257.81 45.72 0)
+      (effects (font (size 1.27 1.27)) hide)
+    )
     (pin "1")
     (pin "2")
@@
       (effects (font (size 1.27 1.27)) hide)
     )
+    (property "LCSC" "C17414" (id 5) (at 252.73 45.72 0)
+      (effects (font (size 1.27 1.27)) hide)
+    )
