File: multicartridge-w27c512/pcb/multicartridge-w27c512.kicad_sch (KiCad schematic)
At the start: 8 parts, among them J1 P2000T_cartridge_edge, SW1 SW_DIP_x02, U1 27C512, U3 74HC00

Commit message: Adding cases
Other:
- note added: "Address line decoding"
- note added: "The lower 12 bits are specified by the P2000T (and the decoder circuit), the upper 2 bits can be set by the user to select the rom."
- note removed: "Adress line decoding"
- note removed: "The lower 12 bits are specified by the P2000T (and the decoder circuit), the upper 5 bits can be set by the user to select the rom."
Changed lines of the file:
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@@
     (effects (font (size 1.27 1.27)) (justify left bottom))
   )
-  (text "Adress line decoding" (at 87.63 20.32 0)
+  (text "Address line decoding" (at 87.63 20.32 0)
     (effects (font (size 1.27 1.27)) (justify left bottom))
   )
-  (text "The lower 12 bits are specified by the\nP2000T (and the decoder circuit), the\nupper 5 bits can be set by the user\nto select the rom."
+  (text "The lower 12 bits are specified by the\nP2000T (and the decoder circuit), the\nupper 2 bits can be set by the user\nto select the rom."
     (at 213.36 34.29 0)
     (effects (font (size 1.27 1.27)) (justify left bottom))
