File: multicartridge/pcb/p2000t-multicartridge/p2000t-multicartridge.kicad_pcb (KiCad board)
At the start: 2 copper layers, 80 x 100 mm, 21 parts, among them J1 P2000T_cartridge_edge, J2 DIPconn, SW1 Soft Reset, U1 SST39SF040, U2 74HC123, U3 74HC00

Commit message: Tuning lay-out multirom cartridge
Parts:
- added REF**: OSHW-Logo2_14.6x12mm_SilkScreen, Symbol:OSHW-Logo2_14.6x12mm_SilkScreen, F.Cu at (79.4, 115.7)
