File: multicartridge-sst39sf010-topbutton/multicartridge-sst39sf010-topbutton/multicartridge-sst39sf010-topbutton.kicad_pcb (KiCad board)
At the start: 2 copper layers, 80 x 105.4 mm, 21 parts, among them J1 P2000T_cartridge_edge, SW1 ~{NMI}, SW2 SW_DIP_x03, U1 SST39SF010, U2 74HC123, U3 74HC00

Commit message: Revising design
Parts:
- added R7: 10k, Resistor_THT:R_Axial_DIN0207_L6.3mm_D2.5mm_P7.62mm_Horizontal, B.Cu at (92.2, 65.9)
- SW2: value SW_DIP_x03 -> SW_DIP_x04; footprint Button_Switch_THT:SW_DIP_SPSTx03_Slide_9.78x9.8mm_W7.62mm_P2.54mm -> Button_Switch_THT:SW_DIP_SPSTx04_Slide_9.78x12.34mm_W7.62mm_P2.54mm
- U1: value SST39SF010 -> SST39SF020
- moved SW2 2.67 mm to (109.3, 56.1)
Connections:
- SW2 pad 4: A14 -> +5V
- SW2 pad 5: A15 -> A14
- SW2 pad 6: A16 -> A15
- U1 pad 30: GND -> A17
Routing:
- net A17: track 0.00 -> 50.8 mm, vias 0 -> 2
- net +5V: track 211.3 -> 213.8 mm
- net A14: track 60.8 -> 62.2 mm
- net GND: track 272.7 -> 271.4 mm
