File: multicartridge-sst39sf010-topbutton/multicartridge-sst39sf010-topbutton/multicartridge-sst39sf010-topbutton.kicad_sch (KiCad schematic)
At the start: 19 parts, among them J1 P2000T_cartridge_edge, SW1 ~{NMI}, SW2 SW_DIP_x03, U1 SST39SF010, U2 74HC123, U3 74HC00

Commit message: Revising design
Parts:
- removed SW2: SW_DIP_x03, Button_Switch_THT:SW_DIP_SPSTx03_Slide_9.78x9.8mm_W7.62mm_P2.54mm, symbol Switch:SW_DIP_x03
- added R7: 10k, Resistor_THT:R_Axial_DIN0207_L6.3mm_D2.5mm_P7.62mm_Horizontal, symbol Device:R
- added SW2: SW_DIP_x04, Button_Switch_THT:SW_DIP_SPSTx04_Slide_9.78x12.34mm_W7.62mm_P2.54mm, symbol Switch:SW_DIP_x04
- U1: value SST39SF010 -> SST39SF020; symbol Memory_Flash:SST39SF010 -> Memory_Flash:SST39SF020
Connections:
- net +5V: now also SW2.1, SW2.2, SW2.3, SW2.4
- net A14: now also SW2.5
- net A15: now also SW2.6
- net A16: now also SW2.7
- net GND: now also R7.1; no longer U1.30 (NC)
- new net A17: R7.2, SW2.8, U1.30 (A17)
